File: Schematic.sch (EAGLE design)
At the start: 105 parts, among them IC1 BQ25180YBGR, IC2 DRV2605YZFR, IC3 BMA423_BMA423, IC9 RT6160AWSC_RT6160AWSC, J1 503480-2400, J2 TC2030-IDC_TC2030-IDC, J4 KH-TYPE-C-16P, Q1 20V/4.2A/52mΩ/1.4W, Q3 SI1308EDL-T1-GE3, U1 NRF52840_QF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

Commit message: Updated file. Fixed issues regarding the schematic.
Parts:
- C2-EP-DR: device InkTime_v5:ESP32_C6_LIBRARY_1_ESP32_WROVER_EAGLE-LTSPICE_CC0402 -> InkTime_v5:NORDIC_NRF_3_CAPACITOR_0603_N
- C20, C21, C6: value 1uF -> 4.7uF
- C25, C33, C39: device InkTime_v5:NORDIC_NRF_3_CAPACITOR_0402_N -> InkTime_v5:NORDIC_NRF_3_CAPACITOR_0603_N
- C27: device InkTime_v5:NORDIC_NRF_3_CAPACITOR_0402_N -> InkTime_v5:NORDIC_NRF_3_CAPACITOR_0201_N
- IC3: value BMA423_BMA423 -> BMA421; ARROW_PART_NUMBER (none) -> BMA421; MANUFACTURER_PART_NUMBER (none) -> BMA421; MOUSER_PART_NUMBER (none) -> 262-BMA421
- L2: device InkTime_v5:NORDIC_NRF_2_INDUCTOR_0402_L -> InkTime_v5:NORDIC_NRF_2_INDUCTOR_0603_N
- renumbered C26 to C1-EP-DR
Connections:
- removed net MU_INT1: IC3.INT1
- removed net MU_INT2: IC3.INT2
- removed net PMIC_IN: IC1.!INT
- net IMU_INT1: now also IC3.INT1
- net IMU_INT2: now also IC3.INT2
- net PMIC_INT: now also IC1.!INT
